Commit message: fix incorrect wheel cord

File: caster_description/urdf/caster.urdf.xacro (robot description, xacro)
@@ -1,7 +1,5 @@
 <?xml version="1.0"?>
 <robot name="caster_robot" xmlns:xacro="http://www.ros.org/wiki/xacro" description="iqr caster robot">
-  <xacro:property name="PI" value="3.1415926535897931" />
-  <xacro:property name="wheel_length" value="0.1143" />
-  <xacro:property name="wheel_radius" value="0.1651" />
+  <xacro:property name="M_PI" value="3.1415926535897931" />
   <xacro:macro name="default_inertial" params="mass">
     <inertial>
@@ -26,9 +24,9 @@
       <xacro:default_inertial mass="0.1" />
     </link>
-    <joint name="support_wheel_${location}_joint" type="continuous">
+    <joint name="support_wheel_${location}_joint" type="fixed">
       <xacro:insert_block name="origin" />
       <parent link="${parent}" />
       <child link="support_wheel_${location}_link" />
-      <axis xyz="0 0 1" />
+      <!-- <axis xyz="0 0 1" /> -->
     </joint>
   </xacro:macro>
@@ -36,6 +34,7 @@
   <xacro:macro name="drive_wheel" params="parent location invert *origin">
     <link name="drive_wheel_${location}_link">
+      <!-- xacro:default_inertial mass="0.1" / -->
       <visual>
-        <origin xyz="0 0 0" rpy="0 0 ${invert*PI}" />
+        <origin xyz="0 0 0" rpy="0 0 ${invert*M_PI}" />
         <geometry>
           <mesh filename="package://caster_description/mesh/drive_wheel.stl" />
@@ -45,5 +44,10 @@
         </material>
       </visual>
-      <!-- xacro:default_inertial mass="0.1" / -->
+      <collision>
+        <origin xyz="0 0 0" rpy="${M_PI/2} 0 0" />
+        <geometry>
+          <cylinder length="0.035" radius="0.075" />
+        </geometry>
+      </collision>
     </link>
     <joint name="drive_wheel_${location}_joint" type="continuous">
@@ -58,5 +62,5 @@
     <link name="ultrasonic_${location}_link">
       <visual>
-        <origin xyz="0 0 0" rpy="0 ${PI/2} 0" />
+        <origin xyz="0 0 0" rpy="0 ${M_PI/2} 0" />
         <geometry>
           <cylinder length="0.01" radius="0.01" />
@@ -89,5 +93,5 @@
   <link name="base_footprint">
     <origin xyz="0 0 0" rpy="0 0 0" />
-    <xacro:default_inertial mass="0.0001" />
+    <!-- <xacro:default_inertial mass="0.0001" /> -->
   </link>
   <joint name="base_footprint_joint" type="fixed">
@@ -134,8 +138,8 @@
   </xacro:ultrasonic>
   <xacro:ultrasonic parent="base_link" location="rear_left">
-    <origin xyz="-0.255 0.055 0.205" rpy="0 0 ${PI}" />
+    <origin xyz="-0.255 0.055 0.205" rpy="0 0 ${M_PI}" />
   </xacro:ultrasonic>
   <xacro:ultrasonic parent="base_link" location="rear_right">
-    <origin xyz="-0.255 -0.055 0.205" rpy="0 0 ${PI}" />
+    <origin xyz="-0.255 -0.055 0.205" rpy="0 0 ${M_PI}" />
   </xacro:ultrasonic>
 </robot>

Commit message: add us, laser, bms and imu to launch

File: caster_description/urdf/caster.urdf.xacro (robot description, xacro)
@@ -78,4 +78,9 @@
     </joint>
   </xacro:macro>
+  <!-- base footprint -->
+  <link name="base_footprint">
+    <origin xyz="0 0 0" rpy="0 0 0" />
+    <!-- <xacro:default_inertial mass="0.0001" /> -->
+  </link>
   <!-- base link -->
   <link name="base_link">
@@ -91,22 +96,22 @@
     <xacro:default_inertial mass="10" />
   </link>
-  <link name="base_footprint">
+  <joint name="base_link_joint" type="fixed">
+    <origin xyz="0 0 0.030" rpy="0 0 0" />
+    <parent link="base_footprint" />
+    <child link="base_link" />
+  </joint>
+  <!-- IMU link -->
+  <link name="imu_link" />
+  <joint name="imu_link_joint" type="fixed">
     <origin xyz="0 0 0" rpy="0 0 0" />
-    <!-- <xacro:default_inertial mass="0.0001" /> -->
-  </link>
-  <joint name="base_footprint_joint" type="fixed">
-    <origin xyz="0 0 -0.030" rpy="0 0 0" />
     <parent link="base_link" />
-    <child link="base_footprint" />
+    <child link="imu_link" />
   </joint>
   <!-- Laser link -->
-  <link name="laser_scan_link">
-    <origin xyz="0 0 0" rpy="0 0 0" />
-    <xacro:default_inertial mass="0.0001" />
-  </link>
-  <joint name="laser_scan_joint" type="fixed">
+  <link name="laser_link" />
+  <joint name="laser_link_joint" type="fixed">
     <origin xyz="0.2301 0 0.147" rpy="0 0 0" />
     <parent link="base_link" />
-    <child link="laser_scan_link" />
+    <child link="laser_link" />
   </joint>
   <!-- Drive wheel link -->

Commit message: add log arg on all launch file

File: caster_description/urdf/caster.urdf.xacro (robot description, xacro)
@@ -137,14 +137,14 @@
   <!-- Ultrasonic link-->
   <xacro:ultrasonic parent="base_link" location="front_left">
-    <origin xyz="0.25 0.075 0.07" rpy="0 0 0" />
+    <origin xyz="0.26248 0.0704 0.0245" rpy="0 0 0.2618" />
   </xacro:ultrasonic>
   <xacro:ultrasonic parent="base_link" location="front_right">
-    <origin xyz="0.25 -0.075 0.07" rpy="0 0 0" />
+    <origin xyz="0.26248 -0.0704 0.0245" rpy="0 0 -0.2618" />
   </xacro:ultrasonic>
   <xacro:ultrasonic parent="base_link" location="rear_left">
-    <origin xyz="-0.255 0.055 0.205" rpy="0 0 ${M_PI}" />
+    <origin xyz="-0.26298 0.0704 0.2095" rpy="0 0 2.8798" />
   </xacro:ultrasonic>
   <xacro:ultrasonic parent="base_link" location="rear_right">
-    <origin xyz="-0.255 -0.055 0.205" rpy="0 0 ${M_PI}" />
+    <origin xyz="-0.26298 -0.0704 0.2095" rpy="0 0 -2.8798" />
   </xacro:ultrasonic>
 </robot>

Commit message: add rplidar, fix dock node problem

File: caster_description/urdf/caster.urdf.xacro (robot description, xacro)
@@ -115,4 +115,11 @@
     <child link="laser_link" />
   </joint>
+  <!-- Laser link 2 (rplidar) -->
+  <link name="laser_link2" />
+  <joint name="laser_link_joint2" type="fixed">
+    <origin xyz="0.01525 0 0.2115" rpy="0 0 0" />
+    <parent link="base_link" />
+    <child link="laser_link2" />
+  </joint>
   <!-- Drive wheel link -->
   <xacro:drive_wheel parent="base_link" invert="0" location="left">

Commit message: fix incorrect rplidar joint yaw angle

File: caster_description/urdf/caster.urdf.xacro (robot description, xacro)
@@ -118,5 +118,5 @@
   <link name="laser_link2" />
   <joint name="laser_link_joint2" type="fixed">
-    <origin xyz="0.01525 0 0.2115" rpy="0 0 0" />
+    <origin xyz="0.01525 0 0.2115" rpy="0 0 ${M_PI}" />
     <parent link="base_link" />
     <child link="laser_link2" />
